File: controller.kicad_sch (KiCad schematic)
At the start: 134 parts, among them IC1 TJA1050T_CM,118, IC2 STSPIN32G4, IC3 AS5600-ASOM, IC4 AS5600-ASOM, J1 XT30XT30PW_MALE, J2 XT30XT30PW_MALE, M1 MOUNT, M2 MOUNT, M3 MOUNT, M4 MOUNT, Q1 TPH1R204PLSOP_ADVANCE_8, Q2 TPH1R204PLSOP_ADVANCE_8, Q3 TPH1R204PLSOP_ADVANCE_8, Q4 TPH1R204PLSOP_ADVANCE_8, Q5 TPH1R204PLSOP_ADVANCE_8, Q6 TPH1R204PLSOP_ADVANCE_8, U4 MAX15062AATA+T

Commit message: Slightly cheaper
Parts:
- removed C20: 1uF, controller:C0603, symbol controller-eagle-import:mfpassives_CAPACITOR_NP_0603
- removed C21: 10uF, controller:C1206, symbol controller-eagle-import:mfpassives_CAPACITOR_NP_1206
- removed C39: 1uF 100V, controller:C0805, symbol controller-eagle-import:mfpassives_CAPACITOR_NP_0805
- removed C56: 1uF, controller:C0402, symbol controller-eagle-import:mfpassives_CAPACITOR_NP_0402
- removed L2: LBM2016T120J, inductor:INDC2016X180N, symbol inductor:LBM2016T120J
- removed U4: MAX15062AATA+T, controller:21-0487A_MXM, symbol controller-eagle-import:MAX15062AATA+T
- added C1, C2: 100uF, Capacitor_SMD:C_1206_3216Metric, symbol Device:C
- added C4: 10uF, controller:C0805, symbol controller-eagle-import:mfpassives_CAPACITOR_NP_0402
- added C5: 0.01uF, controller:C0402, symbol controller-eagle-import:mfpassives_CAPACITOR_NP_0402
- added D14: SS14, DIOM5127X261N, symbol SamacSys:SS14
- added L1: 22uH, Inductor_SMD:L_0805_2012Metric, symbol Device:L
- added R11: 5.6k, controller:R0402, symbol controller-eagle-import:mfpassives_RESISTOR_0402
- added R18: 270, Resistor_SMD:R_0603_1608Metric, symbol Device:R_US
- added R19: 10k, controller:R0402, symbol controller-eagle-import:mfpassives_RESISTOR_0402
- added U1: TPS5430DDAR, Package_SO:TI_SO-PowerPAD-8_ThermalVias, symbol Regulator_Switching:TPS5430DDA
- A0, B0, C0, C55, D33, DA0, DAC0, DB0, DBG1, DBG2, DC0, DG2, M1, M2, M3, M4, R10, TEMP1, TEMP2: now left out of the parts list
- Q2, Q4, Q6: MPN TPH2R506PL,L1Q -> TPH4R50ANH,L1Q(M
- R1, R2: value 560 -> 510
- R22, R23, R24, R25, R26, R27: value 7.5 -> 10
- R5: value 100k 1% -> 100k
- R6: value 4.7k 1% -> 4.7k
- R7, R9: value 10k 1% -> 10k
Connections:
- net +3V3: now also C1.2, C2.2, L1.2, R19.P$2
- net GND: now also C1.1, C2.1, C4.P$1, D14.2, R18.2, U1.6 (GND), U1.9 (GNDPAD)
- net V+: now also C4.P$2, U1.7 (VIN)
- new net: R11.P$1, R19.P$1, U1.4 (VSENSE)
- new net: R11.P$2, R18.1
- new net: C5.P$1, U1.1 (BOOT)
- new net: C5.P$2, D14.1, L1.1, U1.8 (PH)
- no-connect marks 29 -> 28

Commit message: Almost?
Parts:
- removed C1, C2: 100uF, Capacitor_SMD:C_1206_3216Metric, symbol Device:C
- removed C38: 10uF, Capacitor_SMD:C_0402_1005Metric, symbol motor-rescue:C_Small
- removed C4: 10uF, controller:C0805, symbol controller-eagle-import:mfpassives_CAPACITOR_NP_0402
- removed C5: 0.01uF, controller:C0402, symbol controller-eagle-import:mfpassives_CAPACITOR_NP_0402
- removed C64: 100nF, Capacitor_SMD:C_0402_1005Metric, symbol motor-rescue:C_Small
- removed C65: 100nF, controller:C0402, symbol controller-eagle-import:mfpassives_CAPACITOR_NP_0402
- removed D14: SS14, DIOM5127X261N, symbol SamacSys:SS14
- removed L1: 22uH, Inductor_SMD:L_0805_2012Metric, symbol Device:L
- removed R11: 5.6k, controller:R0402, symbol controller-eagle-import:mfpassives_RESISTOR_0402
- removed R15: 1k, controller:R0402, symbol controller-eagle-import:mfpassives_RESISTOR_0402
- removed R18: 270, Resistor_SMD:R_0603_1608Metric, symbol Device:R_US
- removed R19: 10k, controller:R0402, symbol controller-eagle-import:mfpassives_RESISTOR_0402
- removed TEMP1: PAD24AWG_PAD, controller:24AWG_PAD, symbol controller-eagle-import:PAD24AWG_PAD
- removed U1: TPS5430DDAR, Package_SO:TI_SO-PowerPAD-8_ThermalVias, symbol Regulator_Switching:TPS5430DDA
- added C14, C7: 10uF, Capacitor_SMD:C_0402_1005Metric, symbol motor-rescue:C_Small
- added C20: 100nF, Capacitor_SMD:C_0402_1005Metric, symbol motor-rescue:C_Small
- added C21, C39: 100nF, controller:C0402, symbol controller-eagle-import:mfpassives_CAPACITOR_NP_0402
- added C38: 1uF, controller:C0402, symbol controller-eagle-import:mfpassives_CAPACITOR_NP_0402
- added C6: NM1210B224K251CEGN, Capacitor_SMD:C_1210_3225Metric, symbol motor-rescue:C_Small
- added D14: STPS1H100A, Diode_SMD:D_SMA, symbol Device:D_Schottky
- added L2: 18uH/1A, EasyEda2Kicad:IND-SMD_L5.8-W5.2_SCD0503T, symbol Device:L
- added R20, R21, R31, R32: 1.5k, controller:R0402, symbol controller-eagle-import:mfpassives_RESISTOR_0402
- added R28, R29, R33, R34: 22k, controller:R0402, symbol controller-eagle-import:mfpassives_RESISTOR_0402
- added R30, R35: 11k, controller:R0402, symbol controller-eagle-import:mfpassives_RESISTOR_0402
- added U2, U3, U4: Opamp_Dual, symbol Device:Opamp_Dual
- R12, R13: value 1k -> 22k
- R14, R16: value 1k -> 1.5k
- R17: value 1k -> 11k
Connections:
- net +3V3: now also IC2.27 (VDDA), C14.2, C20.2, C21.P$2, C38.P$1, C39.P$1; no longer IC2.64 (REGIN)
- net GND: now also R13.P$2, R17.P$1, C14.1, C20.1, C21.P$1, C38.P$2, C39.P$2, C6.2, C7.2, D14.2 (A), R29.P$2, R30.P$1, R34.P$2, R35.P$1; no longer IC2.27 (VDDA), IC2.61 (VM), IC2.62 (SW), IC2.63 (VCC)
- net SXA_N: now also R14.P$2; no longer R12.P$1
- net SXA_P: now also R16.P$2; no longer R13.P$1
- net SXB_N: now also R21.P$2; no longer R16.P$1
- net SXB_P: now also R20.P$2; no longer R17.P$1
- net SXC_N: now also R32.P$2
- net SXC_P: now also R31.P$2; no longer R14.P$1
- net V+: now also IC2.61 (VM), R12.P$1, C6.1, R28.P$1, R33.P$1
- net PA1: now reaches IC2.14 (PA1)
- net PA1: now also R12.P$2, R13.P$1, R16.P$1, U2.3 (+); no longer R13.P$2
- net PA2: now reaches R17.P$2
- net PA2: now also IC2.15 (PA2), U2.1; no longer IC2.20 (PA7)
- net PC5: now reaches IC2.22 (PC5)
- net PC5: now also R21.P$1, U3.2 (-); no longer R16.P$2
- net PA3: now reaches IC2.16 (PA3)
- net PA3: now also R14.P$1, U2.2 (-); no longer R12.P$2
- net PB2: now reaches IC2.25 (PB2)
- net PB2: now also R32.P$1, U4.2 (-)
- net PA6: now reaches IC2.19 (PA6)
- net PA6: now also R30.P$2, U3.1
- net PB0: now reaches IC2.23 (PB0)
- net PB0: now also R31.P$1, R33.P$2, R34.P$1, U4.3 (+); no longer R14.P$2
- net PB1: now reaches IC2.24 (PB1)
- net PB1: now also R35.P$2, U4.1
- net VOLTAGE DIVIDER HERE: now reaches IC2.52 (SCREF)
- new net: D14.1 (K), IC2.62 (SW), L2.2
- new net: C7.1, IC2.63 (VCC), IC2.64 (REGIN), L2.1
- new net PA7: IC2.20 (PA7), R20.P$1, R28.P$2, R29.P$1, U3.3 (+)
- no-connect marks 28 -> 23
Other:
- moved on the sheet: C16, IC2
