File: pcb/controller.kicad_pcb (KiCad board)
At the start: 4 copper layers, 46 x 53 mm, 142 parts, among them IC1 TJA1050T_CM,118, IC2 STSPIN32G4, IC3 AS5600-ASOM, IC4 AS5600-ASOM, J1 XT30XT30PW_MALE, J2 XT30XT30PW_MALE, M1 MOUNT, M2 MOUNT, M3 MOUNT, M4 MOUNT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

Commit message: PCB changes
Parts:
- removed C10, C8: 0.1uF, controller:C0402
- removed C11: 0.1uF, controller:C0402_NOBORDER
- removed C55: DNP, controller:C0402
- removed C9: 1uF, controller:C0402
- removed D33, DAC0, DBG1, DBG2, DG2: PAD24AWG_PAD, controller:24AWG_PAD
- removed IC1: TJA1050T_CM,118, SamacSys:SOIC127P600X175-8N
- removed IC3, IC4: AS5600-ASOM, SamacSys:SOIC127P600X175-8N
- removed R10: DNP, controller:R0402
- removed R14, R21, R32: 1.5k, controller:R0402
- removed R17, R30, R35: 11k, controller:R0402
- removed R3, R4: 2k, controller:R0402
- added C1: 100nF, controller:C0402, F.Cu at (146.4, 100.0)
- added C2: 0.1uF, controller:C0402, F.Cu at (165.9, 96.2)
- added JP1: SolderJumper_2_Bridged, Jumper:SolderJumper-2_P1.3mm_Bridged_Pad1.0x1.5mm, F.Cu at (169.9, 100.6)
- added JP5: SolderJumper_2_Open, Jumper:SolderJumper-2_P1.3mm_Open_RoundedPad1.0x1.5mm, F.Cu at (168.0, 87.3)
- added JP6: SolderJumper_3_Bridged12, Jumper:SolderJumper-3_P1.3mm_Bridged12_RoundedPad1.0x1.5mm, F.Cu at (168.1, 90.2)
- added JP7: SolderJumper_3_Bridged12, Jumper:SolderJumper-3_P1.3mm_Bridged12_RoundedPad1.0x1.5mm, F.Cu at (168.1, 93.0)
- added R11: 120, controller:R0402, B.Cu at (157.8, 121.3)
- added R15: 10k, controller:R0402, F.Cu at (158.8, 80.6)
- added TH2: 47k, Resistor_SMD:R_0603_1608Metric, F.Cu at (162.5, 82.1)
- added U1: MAX3051, Package_TO_SOT_SMD:TSOT-23-8, F.Cu at (168.2, 96.8)
- added U5: AS5048A, Package_SO:TSSOP-14_4.4x5mm_P0.65mm, B.Cu at (149.3, 97.8)
- C12: value 0.1uF -> 10uF
- C6: value 200nF / 100V -> NM1210B224K251CEGN
- D14: value D_Schottky -> STPS1H100A
- R8: value 47k NTC -> 22k
- moved ABS0 38.0 mm to (129.5, 92.5), turned to 90 degrees
- moved D3 37.7 mm to (149.5, 87.9), turned to 0 degrees
- moved D2 36.2 mm to (149.5, 89.5), turned to 0 degrees
- moved R8 35.0 mm to (157.6, 80.6)
- moved C13 34.3 mm to (163.8, 83.0), turned to 90 degrees
- moved R9 34.3 mm to (165.1, 83.0), turned to 90 degrees
- moved R1 33.1 mm to (146.4, 89.0), turned to 0 degrees
- moved R2 30.9 mm to (145.9, 90.8), turned to 90 degrees
- moved R6 8.82 mm to (161.1, 97.7), turned to -90 degrees
- moved C57 7.70 mm to (160.5, 95.9), turned to 0 degrees
- moved R5 6.62 mm to (159.9, 97.7)
- moved R20 4.70 mm to (154.9, 93.2), turned to 0 degrees
- moved R31 4.48 mm to (157.3, 95.0)
- moved R29 3.64 mm to (154.9, 94.8)
- moved R28 3.17 mm to (152.6, 94.8)
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Connections:
- ABS0 pad 1: +3V3 -> /OUTPUT_PIN
- ABS0 pad 2: /I2C_ABS_SCL -> /UART_TXD
- ABS0 pad 3: /I2C_ABS_SDA -> /UART_RXD
- C12 pad P$1: +3V3 -> +3.3V
- C14 pad 2: +3V3 -> +3.3V
- C19 pad 2: +3V3 -> +3.3V
- C20 pad 2: +3V3 -> +3.3V
- C21 pad P$2: +3V3 -> +3.3V
- C3 pad P$2: +3V3 -> +3.3V
- C38 pad P$1: +3V3 -> +3.3V
- C39 pad P$1: +3V3 -> +3.3V
- D2 pad ANODE: Net-(D2-PadANODE) -> /LED2
- D2 pad CATHODE: /LED2 -> Net-(D2-PadCATHODE)
- D3 pad ANODE: Net-(D3-PadANODE) -> /LED1
- D3 pad CATHODE: /LED1 -> Net-(D3-PadCATHODE)
- ENC0 pad 2: /AS5047_DIR -> /AS5048_CS
- ENC0 pad 4: /AS5047_SCL -> /AS5048_MISO
- ENC0 pad 5: /AS5047_SDA -> /AS5048_SCLK
- ENC0 pad 6: /AS5047_PGO -> /AS5048_MOSI
- IC2 pad 1: +3V3 -> +3.3V
- IC2 pad 15: /PA2 -> unconnected-(IC2-PA2-Pad15)
- IC2 pad 17: /DAC -> unconnected-(IC2-PA4-Pad17)
- IC2 pad 19: /PA6 -> unconnected-(IC2-PA6-Pad19)
- IC2 pad 2: +3V3 -> +3.3V
- IC2 pad 21: /AS5047_SCL -> unconnected-(IC2-PC4-Pad21)
- IC2 pad 24: /PB1 -> unconnected-(IC2-PB1-Pad24)
- IC2 pad 26: +3V3 -> +3.3V
- IC2 pad 27: +3V3 -> +3.3V
- IC2 pad 44: /I2C_ABS_SCL -> /OUTPUT_PIN
- IC2 pad 45: /I2C_ABS_SDA -> /UART_TXD
- IC2 pad 46: unconnected-(IC2-PA10-Pad46) -> /UART_RXD
- IC2 pad 47: /CAN_TX -> Net-(IC2-PA11)
- IC2 pad 48: /CAN_RX -> Net-(IC2-PA12)
- IC2 pad 52: unconnected-(IC2-SCREF-Pad52) -> Net-(IC2-SCREF)
- IC2 pad 53: unconnected-(IC2-PD2-Pad53) -> /AS5048_CS
- IC2 pad 54: unconnected-(IC2-PB3-Pad54) -> /AS5048_SCLK
- IC2 pad 55: /AS5047_PGO -> /AS5048_MISO
- IC2 pad 56: /AS5047_DIR -> /AS5048_MOSI
- IC2 pad 57: unconnected-(IC2-PB6-Pad57) -> /VTEMP_MOT
- IC2 pad 58: unconnected-(IC2-PB7-Pad58) -> /VTEMP_FET
- IC2 pad 59: /VTEMP_FET -> unconnected-(IC2-PB8-Pad59)
- IC2 pad 6: /AS5047_SDA -> unconnected-(IC2-PF0-Pad6)
- IC2 pad 60: /VTEMP_MOT -> unconnected-(IC2-PB9-Pad60)
- NT1 pad 1: /SXB_N -> /PC5
- NT6 pad 1: /SXC_N -> /PB2
- NT8 pad 1: /SXA_N -> /PA3
- R1 pad P$1: +3V3 -> GND
- R1 pad P$2: Net-(D3-PadANODE) -> Net-(D3-PadCATHODE)
- R12 pad P$1: V+ -> +3.3V
- R2 pad P$1: +3V3 -> GND
- R2 pad P$2: Net-(D2-PadANODE) -> Net-(D2-PadCATHODE)
- R28 pad P$1: V+ -> +3.3V
- R33 pad P$1: V+ -> +3.3V
- R8 pad P$1: +3V3 -> Net-(IC2-SCREF)
- R8 pad P$2: /VTEMP_FET -> +3.3V
- SWD0 pad 6: +3V3 -> +3.3V
Routing:
- net +3V3: track 176.2 -> 0.00 mm, vias 13 -> 0
- net GND: track 186.3 -> 89.0 mm, vias 108 -> 114
- net /LED1: track 83.8 -> 1.83 mm, vias 2 -> 0
- net /LED2: track 82.1 -> 2.10 mm, vias 2 -> 0
- net /AS5047_SCL: track 55.4 -> 0.00 mm, vias 2 -> 0
- net /AS5048_CS: track 0.00 -> 54.4 mm, vias 0 -> 4
- net +3.3V: track 0.00 -> 54.0 mm, vias 0 -> 9
- net /AS5047_SDA: track 53.4 -> 0.00 mm, vias 2 -> 0
- net /AS5047_PGO: track 50.6 -> 0.00 mm, vias 2 -> 0
- net /AS5047_DIR: track 47.1 -> 0.00 mm, vias 3 -> 0
- net /AS5048_SCLK: track 0.00 -> 43.7 mm, vias 0 -> 4
- net /AS5048_MISO: track 0.00 -> 43.7 mm, vias 0 -> 4
- net /VTEMP_FET: track 54.7 -> 13.0 mm
- net /OUTPUT_PIN: track 0.00 -> 39.9 mm, vias 0 -> 2
- net /UART_TXD: track 0.00 -> 39.5 mm, vias 0 -> 2
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- added copper zone on In2.Cu, net +3.3V
- removed copper zone on In2.Cu, net +3V3

Commit message: can_monitor - ability to scroll messages - use can send for extended id
main.cpp
- ignore bitrate switching, not needed.
- add can debug messages for all SimpleFOC serial messages
- support extended CAN messages
- reduce current limit
- motor monitoring through CAN

Update schematic and PCB to latest version
Parts:
- removed R20: 1.5k, controller:R0402
- added R10: 1.5k 1%, Resistor_SMD:R_0402_1005Metric, F.Cu at (157.2, 93.9)
- added R14: 11k 1%, Resistor_SMD:R_0402_1005Metric, F.Cu at (156.8, 92.5)
- added R17: 11k 1%, Resistor_SMD:R_0402_1005Metric, F.Cu at (154.6, 92.5)
- added R18: 11k 1%, Resistor_SMD:R_0402_1005Metric, F.Cu at (150.3, 91.3)
- added R19: 1.5k 1%, Resistor_SMD:R_0402_1005Metric, F.Cu at (154.6, 94.5)
- added R3: 1.5k 1%, Resistor_SMD:R_0402_1005Metric, F.Cu at (154.6, 93.5)
- added R4: 1.5k 1%, Resistor_SMD:R_0402_1005Metric, F.Cu at (148.8, 92.6)
- C1, C12, C13, C15, C16, C17, C18, C2, C21, C3, C38, C39, C57: footprint controller:C0402 -> Capacitor_SMD:C_0402_1005Metric
- C22, C23, C24, C25, C26, C27, C28, C29, C30, C31, C32, C33, C34, C36, C37, C61, C63: footprint controller:C1206 -> Capacitor_SMD:C_1206_3216Metric
- C35: footprint controller:C1206_NOBORDER -> Capacitor_SMD:C_1206_3216Metric
- C40, C41, C42, C43, C44, C45, C46, C47, C48, C49, C50, C51, C52, C53, C54: footprint controller:C1206_NOCREAM -> Capacitor_SMD:C_1206_3216Metric
- D2, D3: footprint controller:LED0603 -> LED_SMD:LED_0603_1608Metric
- M1, M2, M3, M4: footprint MountingHole:MountingHole_2.7mm_M2.5_DIN965_Pad -> MountingHole:MountingHole_3.2mm_M3_DIN965_Pad
- R1, R11, R12, R15, R2, R22, R23, R24, R25, R26, R27, R5, R6, R7, R8, R9: footprint controller:R0402 -> Resistor_SMD:R_0402_1005Metric
- R13, R28, R29, R33, R34: value 22k -> 22k 1%; footprint controller:R0402 -> Resistor_SMD:R_0402_1005Metric
- R16, R31: value 1.5k -> 1.5k 1%; footprint controller:R0402 -> Resistor_SMD:R_0402_1005Metric
- RA0, RB0, RC0: value 0.5mOhm 1% 2W -> 5mOhm 1% 2W; footprint controller:M1206 -> Resistor_SMD:R_1206_3216Metric
- moved R16 8.09 mm to (147.1, 92.8)
- moved R6 6.43 mm to (154.8, 96.1), turned to 180 degrees
- moved R5 6.01 mm to (153.9, 97.0), turned to 180 degrees
- moved C57 4.96 mm to (155.8, 97.3)
- moved R29 2.26 mm to (152.7, 94.6), turned to 180 degrees
- moved R33 1.98 mm to (156.7, 95.5)
- moved R9 1.59 mm to (164.4, 84.5), turned to 0 degrees
- moved R31 1.42 mm to (156.3, 93.9), turned to -90 degrees
- moved C3 0.83 mm to (158.7, 92.6)
- moved R28 0.82 mm to (152.7, 95.6)
- moved R34 0.53 mm to (156.8, 96.4)
- moved C21 0.45 mm to (160.5, 93.1)
- moved D2 0.22 mm to (149.7, 89.4)
- moved C17 0.19 mm to (162.7, 88.3)
- moved D3 0.19 mm to (149.7, 87.8)
Connections:
- IC2 pad 15: unconnected-(IC2-PA2-Pad15) -> /PA2
- IC2 pad 19: unconnected-(IC2-PA6-Pad19) -> /PA6
- IC2 pad 24: unconnected-(IC2-PB1-Pad24) -> /PB1
- NT1 pad 1: /PC5 -> /SXB_N
- NT6 pad 1: /PB2 -> /SXC_N
- NT8 pad 1: /PA3 -> /SXA_N
Routing:
- net /PA3: track 20.7 -> 3.55 mm
- net /PB2: track 18.7 -> 2.38 mm
- net /PC5: track 18.0 -> 2.06 mm
- net /SXA_N: track 0.00 -> 15.9 mm
- net /SXB_N: track 0.00 -> 14.8 mm
- net /SXC_N: track 0.00 -> 14.0 mm
- net /SXA_P: track 6.14 -> 14.9 mm
- net /PA1: track 16.4 -> 7.89 mm
- net GND: track 89.0 -> 95.3 mm, vias 114 -> 113
- net /VBAT_SENSE: track 13.5 -> 7.52 mm
- net /CAN_N: track 69.1 -> 63.2 mm
- net +3.3V: track 54.0 -> 59.2 mm, vias 9 -> 10
- net V+: track 38.3 -> 34.3 mm
- net Net-(D2-PadCATHODE): track 3.15 -> 0.00 mm
- net Net-(D2-K): track 0.00 -> 2.99 mm
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